Commit message: feat: add FastAPI web server and ROS 2 bridge for autonomous AMR fleet control

File: src/ackermann_car_sim/urdf/ackermann_car.urdf.xacro (robot description, xacro)
@@ -2,5 +2,5 @@
 <robot name="ackermann_car" xmlns:xacro="http://www.ros.org/wiki/xacro">
   <!-- ==================== PARAMETERS ==================== -->
-  <xacro:property name="wheelbase" value="0.20"/>
+  <xacro:property name="wheelbase" value="0.15"/>
   <xacro:property name="track_width" value="0.18"/>
   <xacro:property name="wheel_radius" value="0.035"/>
@@ -158,6 +158,6 @@
     <parent link="base_link"/>
     <child link="lidar_link"/>
-    <!-- LiDAR öne alındı: ön engelleri daha erken algılar (K-3 düzeltmesi) -->
-    <origin xyz="${chassis_length/2 - 0.02} 0 ${chassis_height + 0.04}" rpy="0 0 0"/>
+    <!-- LiDAR şasinin tam merkezinde (köşegenlerin kesişim noktası) -->
+    <origin xyz="0 0 ${chassis_height + 0.04}" rpy="0 0 0"/>
   </joint>
   <!-- ==================== INTEL REALSENSE CAMERA ==================== -->
